File: pcbs/socket_shield/socket_shield/socket_shield.kicad_sch (KiCad schematic)
At the start: 17 parts, among them J1 Power, J2 PWM, J3 Analog, J4 PWM, J5 Analog, J6 Communication, J7 Digital

Commit message: increase hole sizes for socket
Parts:
- U1: footprint Package_DIP:DIP-28_W15.24mm_Socket_LongPads -> customs-fp:DIP-28_600_ELL
Changed lines of the file:
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@@
 			)
 		)
-		(property "Footprint" "Package_DIP:DIP-28_W15.24mm_Socket_LongPads"
+		(property "Footprint" "customs-fp:DIP-28_600_ELL"
 			(at 133.35 31.75 0)
 			(effects

Commit message: add id pins at designate the socket shield as id 0x01
Connections:
- net 49 is gone; now on net GND: J7.8 (Pin_8)
- net *44 renamed id5
- net *45 renamed id4
- net *46 renamed id3
- net 42 renamed id7
- net 43 renamed id6
- net 47 renamed id2
- net 48 renamed id1
Changed lines of the file:
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@@
 		)
 	)
-	(label "*44"
+	(label "id5"
 		(at 39.37 109.22 270)
 		(effects
@@
 		)
 	)
-	(label "47"
+	(label "id2"
 		(at 36.83 142.24 90)
 		(effects
@@
 		)
 	)
-	(label "*45"
+	(label "id4"
 		(at 39.37 142.24 90)
 		(effects
@@
 		)
 	)
-	(label "42"
+	(label "id7"
 		(at 41.91 109.22 270)
 		(effects
@@
 		)
 	)
-	(label "*46"
+	(label "id3"
 		(at 36.83 109.22 270)
 		(effects
@@
 		)
 	)
-	(label "49"
+	(label "id0"
 		(at 34.29 142.24 90)
 		(effects
@@
 		)
 	)
-	(label "43"
+	(label "id6"
 		(at 41.91 142.24 90)
 		(effects
@@
 		)
 	)
-	(label "48"
+	(label "id1"
 		(at 34.29 109.22 270)
 		(effects
@@
 					(unit 1)
 				)
+			)
+		)
+	)
+	(symbol
+		(lib_id "power:GND")
+		(at 34.29 142.24 0)
+		(unit 1)
+		(exclude_from_sim no)
+		(in_bom yes)
+		(on_board yes)
+		(dnp no)
+		(property "Reference" "#PWR014"
+			(at 34.29 148.59 0)
+			(effects
+				(font
+					(size 1.27 1.27)
+				)
+				(hide yes)
+			)
+		)
+		(property "Value" "GND"
+			(at 34.4043 146.5644 0)
+			(effects
+				(font
+					(size 1.27 1.27)
+				)
+			)
+		)
+		(property "Footprint" ""
+			(at 34.29 142.24 0)
+			(effects
+				(font
+					(size 1.27 1.27)
+				)
+			)
+		)
+		(property "Datasheet" ""
+			(at 34.29 142.24 0)
+			(effects
+				(font
+					(size 1.27 1.27)
+				)
+			)
+		)
+		(property "Description" "Power symbol creates a global label with name \"GND\" , ground"
+			(at 34.29 142.24 0)
+			(effects
+				(font
+					(size 1.27 1.27)
+				)
+				(hide yes)
+			)
+		)
+		(pin "1"
+		)
+		(instances
+			(project "socket_shield"
+				(path "/e63e39d7-6ac0-4ffd-8aa3-1841a4541b55"
+					(reference "#PWR014")
+					(unit 1)
+				)
