File: pcbs/socket_shield/socket_shield.kicad_sch (KiCad schematic)
At the start: 17 parts, among them J1 Power, J2 PWM, J3 Analog, J4 PWM, J5 Analog, J6 Communication, J7 Digital

Commit message: move PCB
Parts:
- removed J4: PWM, Connector_PinSocket_2.54mm:PinSocket_1x08_P2.54mm_Vertical, symbol Connector_Generic:Conn_01x08
- removed J6: Communication, Connector_PinSocket_2.54mm:PinSocket_1x08_P2.54mm_Vertical, symbol Connector_Generic:Conn_01x08
- U1: value ~ -> (none)
Connections:
- net GND: now also R4.2, R5.2, R6.2; no longer D1.1 (K), D2.1 (K), D3.1 (K)
- net LED_active: now also D1.2 (A); no longer R4.1
- net LED_error: now also D3.2 (A); no longer R6.1
- net LED_write: now also D2.2 (A); no longer R5.1
- new net: D2.1 (K), R5.1
- new net: D3.1 (K), R6.1
- new net: D1.1 (K), R4.1
- no-connect marks 1 -> 30
Other:
- moved on the sheet: R4, R5, R6
